File: kicad_ci_test.kicad_sch (KiCad schematic)
At the start: 4 parts, among them J1 Conn_01x02_Socket, J2 Conn_01x02_Socket

Commit message: test
Parts:
- R1: value 100 -> 200
Changed lines of the file:
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@@
 (kicad_sch
-	(version 20231120)
+	(version 20250114)
 	(generator "eeschema")
-	(generator_version "8.0")
+	(generator_version "9.0")
 	(paper "A4")
 	(title_block
@@
 			)
 		)
-		(property "Value" "100"
+		(property "Value" "200"
 			(at 101.6 64.3636 90)
 			(effects
@@
 		)
 	)
+	(embedded_fonts no)
 )
